File: Hardware/Production/RGB_PMOLED_0.6IN-Panel.brd (EAGLE design)
At the start: 99.8 x 102.4 mm, 411 parts, among them Q1 310mA/60V/1.6Ω, Q2 310mA/60V/1.6Ω, Q3 310mA/60V/1.6Ω, Q4 310mA/60V/1.6Ω, Q5 310mA/60V/1.6Ω, Q6 310mA/60V/1.6Ω, Q7 310mA/60V/1.6Ω, Q8 310mA/60V/1.6Ω, Q9 310mA/60V/1.6Ω, U1 UG-6464TDDBG01-FLD, U10 3.3V, U11 TXB0104, U12 UG-6464TDDBG01-FLD, U13 AP3012, U14 3.3V, U15 TXB0104, U16 UG-6464TDDBG01-FLD, U17 AP3012, U18 3.3V, U19 TXB0104, U2 AP3012, U20 UG-6464TDDBG01-FLD, U21 AP3012, U22 3.3V, U23 TXB0104, U24 UG-6464TDDBG01-FLD, U25 AP3012, U26 3.3V, U27 TXB0104, U28 UG-6464TDDBG01-FLD, U29 AP3012, U3 3.3V, U30 3.3V, U31 TXB0104, U32 UG-6464TDDBG01-FLD, U33 AP3012, U34 3.3V, U35 TXB0104, U36 UG-6464TDDBG01-FLD, U4 TXB0104, U5 AP3012, U6 3.3V, U7 TXB0104, U8 UG-6464TDDBG01-FLD, U9 AP3012

Commit message: Cleaned up documentation
Parts:
- L1, L2, L3, L4, L5, L6, L7, L8, L9: device SparkFun-Coils:INDUCTOR_3X3 -> SparkFun-Coils:INDUCTOR_4.7UH
- U1, U12, U16, U20, U24, U28, U32, U36, U8: value UG-6464TDDBG01-FLD -> UG-6464TDDBG01; device RGB_OLED:UG-6464TDDBG01-FOLDED -> RGB_OLED:AMPHENOL_10051922-2010ELF
- moved U28 10.3 mm to (11.4, 84.8), turned to 180 degrees
- moved U32 10.3 mm to (37.3, 84.8), turned to 180 degrees
- moved U36 10.3 mm to (63.2, 84.8), turned to 180 degrees
- moved U16 9.09 mm to (11.4, 53.8), turned to 180 degrees
- moved U20 9.09 mm to (37.3, 53.8), turned to 180 degrees
- moved U24 9.09 mm to (63.2, 53.8), turned to 180 degrees
- moved U1 7.85 mm to (11.4, 22.9), turned to 180 degrees
- moved U12 7.85 mm to (63.2, 22.9), turned to 180 degrees
- moved U8 7.85 mm to (37.3, 22.9), turned to 180 degrees
- moved E$1 3.81 mm to (9.40, 94.6)
- moved E$2 3.81 mm to (9.40, 94.6)
- moved E$3 3.81 mm to (65.3, 94.6)
- moved E$4 3.81 mm to (65.3, 94.6)
- moved FD25 3.81 mm to (1.27, 91.2)
- moved FD28 3.81 mm to (1.27, 91.2)
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Connections:
- net GND: now also U1.P$21, U1.P$22
- net GND1: now also U8.P$21, U8.P$22
- net GND2: now also U12.P$21, U12.P$22
- net GND3: now also U16.P$21, U16.P$22
- net GND4: now also U20.P$21, U20.P$22
- net GND5: now also U24.P$21, U24.P$22
- net GND6: now also U28.P$21, U28.P$22
- net GND7: now also U32.P$21, U32.P$22
- net GND8: now also U36.P$21, U36.P$22
Routing:
- net GND7: track 83.7 -> 71.3 mm
- net GND6: track 83.7 -> 71.3 mm
- net GND8: track 83.7 -> 71.3 mm
- net GND4: track 83.7 -> 71.3 mm
- net GND3: track 83.7 -> 71.3 mm
- net GND: track 83.7 -> 71.3 mm
- net GND5: track 83.7 -> 71.3 mm
- net GND1: track 83.7 -> 71.3 mm
- net GND2: track 83.7 -> 71.3 mm
- net N$24: track 17.7 -> 8.72 mm
- net N$20: track 17.7 -> 8.72 mm
- net N$16: track 17.7 -> 8.72 mm
- net N$7: track 17.7 -> 8.72 mm
- net N$12: track 17.7 -> 8.72 mm
- net N$5: track 17.7 -> 8.72 mm
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Other:
- board size 99.8 x 102.4 mm -> 99.8 x 106.2 mm
- board text added: "X02"
- board text removed: "X01"
